File: kicad/stm32l053c.sch (KiCad schematic (older format))
At the start: 30 parts, among them P1 SWD, SW1 SW_PUSH, SW2 SW_PUSH, SW3 SW_PUSH, U1 STM32L053C8_LQFP48, U2 TLV61225, Y1 Crystal

Commit message: Footprints for buttons & zebra
Parts:
- added R7: 0, Resistors_SMD:R_0805_HandSoldering, symbol R
- DS1: footprint (none) -> theapi:ZEBRA-12
- Q1: renamed from Q?; footprint (none) -> TO_SOT_Packages_SMD:SOT-23_Handsoldering
- SW1, SW2, SW3: footprint (none) -> theapi:SW_PCB
- W1: renamed from W?; value TEST_1P -> TEST_VDD; footprint (none) -> Measurement_Points:Measurement_Point_Round-SMD-Pad_Big
Connections:
- wire segments 80 -> 82
Changed lines of the file:
@@
 encoding utf-8
 Sheet 1 1
-Title ""
+Title "Kitchen Timer"
 Date ""
-Rev ""
-Comp ""
+Rev "v1.0"
+Comp "theapi"
 Comment1 ""
 Comment2 ""
@@
 $EndDescr
 $Comp
-L Earth #PWR26
+L Earth #PWR01
 U 1 1 58021BE1
 P 4900 7200
-F 0 "#PWR26" H 4900 6950 50  0001 C CNN
+F 0 "#PWR01" H 4900 6950 50  0001 C CNN
 F 1 "Earth" H 4900 7050 50  0001 C CNN
 F 2 "" H 4900 7200 50  0000 C CNN
@@
 $EndComp
 $Comp
-L VDD #PWR24
+L VDD #PWR02
 U 1 1 58021C2A
 P 4900 6900
-F 0 "#PWR24" H 4900 6750 50  0001 C CNN
+F 0 "#PWR02" H 4900 6750 50  0001 C CNN
 F 1 "VDD" H 4900 7050 50  0000 C CNN
 F 2 "" H 4900 6900 50  0000 C CNN
@@
 $EndComp
 $Comp
-L GNDA #PWR18
+L GNDA #PWR03
 U 1 1 58021F75
 P 5100 6300
-F 0 "#PWR18" H 5100 6050 50  0001 C CNN
+F 0 "#PWR03" H 5100 6050 50  0001 C CNN
 F 1 "GNDA" H 5100 6150 50  0000 C CNN
 F 2 "" H 5100 6300 50  0000 C CNN
@@
 $EndComp
 $Comp
-L Earth #PWR19
+L Earth #PWR04
 U 1 1 58021F89
 P 5600 6300
-F 0 "#PWR19" H 5600 6050 50  0001 C CNN
+F 0 "#PWR04" H 5600 6050 50  0001 C CNN
 F 1 "Earth" H 5600 6150 50  0001 C CNN
 F 2 "" H 5600 6300 50  0000 C CNN
@@
 $EndComp
 $Comp
-L GNDA #PWR15
+L GNDA #PWR05
 U 1 1 58022154
 P 5150 5800
-F 0 "#PWR15" H 5150 5550 50  0001 C CNN
+F 0 "#PWR05" H 5150 5550 50  0001 C CNN
 F 1 "GNDA" H 5150 5650 50  0000 C CNN
 F 2 "" H 5150 5800 50  0000 C CNN
@@
 $EndComp
 $Comp
-L Earth #PWR16
+L Earth #PWR06
 U 1 1 580221FA
 P 5650 5800
-F 0 "#PWR16" H 5650 5550 50  0001 C CNN
+F 0 "#PWR06" H 5650 5550 50  0001 C CNN
 F 1 "Earth" H 5650 5650 50  0001 C CNN
 F 2 "" H 5650 5800 50  0000 C CNN
@@
 $EndComp
 $Comp
-L VDD #PWR1
+L VDD #PWR07
 U 1 1 5802295B
 P 5450 1050
-F 0 "#PWR1" H 5450 900 50  0001 C CNN
+F 0 "#PWR07" H 5450 900 50  0001 C CNN
 F 1 "VDD" H 5450 1200 50  0000 C CNN
 F 2 "" H 5450 1050 50  0000 C CNN
@@
 $EndComp
 $Comp
-L Earth #PWR4
+L Earth #PWR08
 U 1 1 5803310F
 P 4800 1800
-F 0 "#PWR4" H 4800 1550 50  0001 C CNN
+F 0 "#PWR08" H 4800 1550 50  0001 C CNN
 F 1 "Earth" H 4800 1650 50  0001 C CNN
 F 2 "" H 4800 1800 50  0000 C CNN
@@
 $EndComp
 $Comp
-L Earth #PWR3
+L Earth #PWR09
 U 1 1 580369A9
 P 2150 1400
-F 0 "#PWR3" H 2150 1150 50  0001 C CNN
+F 0 "#PWR09" H 2150 1150 50  0001 C CNN
 F 1 "Earth" H 2150 1250 50  0001 C CNN
 F 2 "" H 2150 1400 50  0000 C CNN
@@
 NRST
 $Comp
-L VDD #PWR2
+L VDD #PWR010
 U 1 1 5803734F
 P 1650 1200
-F 0 "#PWR2" H 1650 1050 50  0001 C CNN
+F 0 "#PWR010" H 1650 1050 50  0001 C CNN
 F 1 "VDD" H 1650 1350 50  0000 C CNN
 F 2 "" H 1650 1200 50  0000 C CNN
@@
 $EndComp
 $Comp
-L Earth #PWR27
+L Earth #PWR011
 U 1 1 5803BDC8
 P 5950 7200
-F 0 "#PWR27" H 5950 6950 50  0001 C CNN
+F 0 "#PWR011" H 5950 6950 50  0001 C CNN
 F 1 "Earth" H 5950 7050 50  0001 C CNN
 F 2 "" H 5950 7200 50  0000 C CNN
@@
 $EndComp
 $Comp
-L Earth #PWR13
+L Earth #PWR012
 U 1 1 58065816
 P 6550 5400
-F 0 "#PWR13" H 6550 5150 50  0001 C CNN
+F 0 "#PWR012" H 6550 5150 50  0001 C CNN
 F 1 "Earth" H 6550 5250 50  0001 C CNN
 F 2 "" H 6550 5400 50  0000 C CNN
@@
 $EndComp
 $Comp
-L Earth #PWR14
+L Earth #PWR013
 U 1 1 5806680D
 P 3600 5700
-F 0 "#PWR14" H 3600 5450 50  0001 C CNN
+F 0 "#PWR013" H 3600 5450 50  0001 C CNN
 F 1 "Earth" H 3600 5550 50  0001 C CNN
 F 2 "" H 3600 5700 50  0000 C CNN
@@
 $EndComp
 $Comp
-L Earth #PWR5
+L Earth #PWR014
 U 1 1 58077163
 P 9600 2300
-F 0 "#PWR5" H 9600 2050 50  0001 C CNN
+F 0 "#PWR014" H 9600 2050 50  0001 C CNN
 F 1 "Earth" H 9600 2150 50  0001 C CNN
 F 2 "" H 9600 2300 50  0000 C CNN
@@
 F 0 "DS1" V 9500 4200 60  0000 C CNN
 F 1 "LCD_KITCHEN_TIMER" H 9500 4050 60  0000 C CNN
-F 2 "" H 9500 3950 60  0001 C CNN
+F 2 "theapi:ZEBRA-12" H 9500 3950 60  0001 C CNN
 F 3 "" H 9500 3950 60  0000 C CNN
 	1    9500 3950
@@
 $EndComp
 $Comp
-L +BATT #PWR21
+L +BATT #PWR015
 U 1 1 584F2368
 P 850 6750
-F 0 "#PWR21" H 850 6600 50  0001 C CNN
+F 0 "#PWR015" H 850 6600 50  0001 C CNN
 F 1 "+BATT" H 850 6890 50  0000 C CNN
 F 2 "" H 850 6750 50  0000 C CNN
@@
 Connection ~ 1600 6750
 Wire Wire Line
-	2600 6550 3550 6550
+	2600 6550 3100 6550
 Connection ~ 2850 6550
 Wire Wire Line
@@
 Connection ~ 2700 6550
 $Comp
-L Earth #PWR23
+L Earth #PWR016
 U 1 1 584F287E
 P 2850 6850
-F 0 "#PWR23" H 2850 6600 50  0001 C CNN
+F 0 "#PWR016" H 2850 6600 50  0001 C CNN
 F 1 "Earth" H 2850 6700 50  0001 C CNN
 F 2 "" H 2850 6850 50  0000 C CNN
@@
 $EndComp
 $Comp
-L Earth #PWR22
+L Earth #PWR017
 U 1 1 584F28E3
 P 1700 6850
-F 0 "#PWR22" H 1700 6600 50  0001 C CNN
+F 0 "#PWR017" H 1700 6600 50  0001 C CNN
 F 1 "Earth" H 1700 6700 50  0001 C CNN
 F 2 "" H 1700 6850 50  0000 C CNN
@@
 $EndComp
 $Comp
-L Earth #PWR25
+L Earth #PWR018
 U 1 1 584F2924
 P 1250 7050
-F 0 "#PWR25" H 1250 6800 50  0001 C CNN
+F 0 "#PWR018" H 1250 6800 50  0001 C CNN
 F 1 "Earth" H 1250 6900 50  0001 C CNN
 F 2 "" H 1250 7050 50  0000 C CNN
@@
 $EndComp
 $Comp
-L VDD #PWR20
+L VDD #PWR019
 U 1 1 584F2A51
-P 3550 6550
-F 0 "#PWR20" H 3550 6400 50  0001 C CNN
-F 1 "VDD" H 3550 6700 50  0000 C CNN
-F 2 "" H 3550 6550 50  0000 C CNN
-F 3 "" H 3550 6550 50  0000 C CNN
-	1    3550 6550
-	1    0    0    -1
-$EndComp
-Text Notes 3650 6550 0    60   ~ 0
+P 3700 6400
+F 0 "#PWR019" H 3700 6250 50  0001 C CNN
+F 1 "VDD" H 3700 6550 50  0000 C CNN
+F 2 "" H 3700 6400 50  0000 C CNN
+F 3 "" H 3700 6400 50  0000 C CNN
+	1    3700 6400
+	1    0    0    -1
+$EndComp
+Text Notes 3800 6350 0    60   ~ 0
 3V3
 Text Notes 750  6850 0    60   ~ 0
@@
 F 0 "SW1" H 1850 2960 50  0000 C CNN
 F 1 "SW_PUSH" H 1700 2770 50  0000 C CNN
-F 2 "" H 1700 2850 50  0001 C CNN
+F 2 "theapi:SW_PCB" H 1700 2850 50  0001 C CNN
 F 3 "" H 1700 2850 50  0000 C CNN
 	1    1700 2850
@@
 $EndComp
 $Comp
-L VDD #PWR6
+L VDD #PWR020
 U 1 1 585069C3
 P 1300 2700
-F 0 "#PWR6" H 1300 2550 50  0001 C CNN
+F 0 "#PWR020" H 1300 2550 50  0001 C CNN
 F 1 "VDD" H 1300 2850 50  0000 C CNN
 F 2 "" H 1300 2700 50  0000 C CNN
@@
 F 0 "SW2" H 1850 3560 50  0000 C CNN
 F 1 "SW_PUSH" H 1700 3370 50  0000 C CNN
-F 2 "" H 1700 3450 50  0001 C CNN
+F 2 "theapi:SW_PCB" H 1700 3450 50  0001 C CNN
 F 3 "" H 1700 3450 50  0000 C CNN
 	1    1700 3450
@@
 $EndComp
 $Comp
-L VDD #PWR8
+L VDD #PWR021
 U 1 1 58506BE4
 P 1300 3300
-F 0 "#PWR8" H 1300 3150 50  0001 C CNN
+F 0 "#PWR021" H 1300 3150 50  0001 C CNN
 F 1 "VDD" H 1300 3450 50  0000 C CNN
 F 2 "" H 1300 3300 50  0000 C CNN
@@
 F 0 "SW3" H 1850 4160 50  0000 C CNN
 F 1 "SW_PUSH" H 1700 3970 50  0000 C CNN
-F 2 "" H 1700 4050 50  0001 C CNN
+F 2 "theapi:SW_PCB" H 1700 4050 50  0001 C CNN
 F 3 "" H 1700 4050 50  0000 C CNN
 	1    1700 4050
@@
 $EndComp
 $Comp
-L VDD #PWR10
+L VDD #PWR022
 U 1 1 58506C86
 P 1300 3900
-F 0 "#PWR10" H 1300 3750 50  0001 C CNN
+F 0 "#PWR022" H 1300 3750 50  0001 C CNN
 F 1 "VDD" H 1300 4050 50  0000 C CNN
 F 2 "" H 1300 3900 50  0000 C CNN
@@
 	2450 2850 3000 2850
 $Comp
-L Earth #PWR7
+L Earth #PWR023
 U 1 1 5851A35F
 P 2450 3150
-F 0 "#PWR7" H 2450 2900 50  0001 C CNN
+F 0 "#PWR023" H 2450 2900 50  0001 C CNN
 F 1 "Earth" H 2450 3000 50  0001 C CNN
 F 2 "" H 2450 3150 50  0000 C CNN
@@
 $EndComp
 $Comp
-L Earth #PWR9
+L Earth #PWR024
 U 1 1 5851A4F4
 P 2450 3750
-F 0 "#PWR9" H 2450 3500 50  0001 C CNN
+F 0 "#PWR024" H 2450 3500 50  0001 C CNN
 F 1 "Earth" H 2450 3600 50  0001 C CNN
 F 2 "" H 2450 3750 50  0000 C CNN
@@
 $EndComp
 $Comp
-L Earth #PWR11
+L Earth #PWR025
 U 1 1 5851A54D
 P 2450 4350
-F 0 "#PWR11" H 2450 4100 50  0001 C CNN
+F 0 "#PWR025" H 2450 4100 50  0001 C CNN
 F 1 "Earth" H 2450 4200 50  0001 C CNN
 F 2 "" H 2450 4350 50  0000 C CNN
@@
 	8600 5650 8200 5650
 $Comp
-L Earth #PWR17
+L Earth #PWR026
 U 1 1 5851B22D
 P 9300 5850
-F 0 "#PWR17" H 9300 5600 50  0001 C CNN
+F 0 "#PWR026" H 9300 5600 50  0001 C CNN
 F 1 "Earth" H 9300 5700 50  0001 C CNN
 F 2 "" H 9300 5850 50  0000 C CNN
@@
 $EndComp
 $Comp
-L VDD #PWR12
+L VDD #PWR027
 U 1 1 5851B377
 P 9300 5150
-F 0 "#PWR12" H 9300 5000 50  0001 C CNN
+F 0 "#PWR027" H 9300 5000 50  0001 C CNN
 F 1 "VDD" H 9300 5300 50  0000 C CNN
 F 2 "" H 9300 5150 50  0000 C CNN
@@
 $EndComp
 $Comp
-L TEST_1P W?
+L TEST_1P W1
 U 1 1 58557FAC
-P 3200 6400
-F 0 "W?" H 3200 6670 50  0000 C CNN
-F 1 "TEST_1P" H 3200 6600 50  0000 C CNN
-F 2 "" H 3400 6400 50  0000 C CNN
-F 3 "" H 3400 6400 50  0000 C CNN
-	1    3200 6400
-	1    0    0    -1
-$EndComp
-Wire Wire Line
-	3200 6400 3200 6550
-Connection ~ 3200 6550
-$Comp
-L Q_NMOS_GSD Q?
+P 3400 6400
+F 0 "W1" H 3400 6670 50  0000 C CNN
+F 1 "TEST_VDD" H 3400 6600 50  0000 C CNN
+F 2 "Measurement_Points:Measurement_Point_Round-SMD-Pad_Big" H 3600 6400 50  0001 C CNN
+F 3 "" H 3600 6400 50  0000 C CNN
+	1    3400 6400
+	1    0    0    -1
+$EndComp
+$Comp
+L Q_NMOS_GSD Q1
 U 1 1 585590EB
 P 9200 5650
-F 0 "Q?" H 9500 5700 50  0000 R CNN
+F 0 "Q1" H 9500 5700 50  0000 R CNN
 F 1 "Q_NMOS_GSD" H 9850 5600 50  0000 R CNN
-F 2 "" H 9400 5750 50  0000 C CNN
+F 2 "TO_SOT_Packages_SMD:SOT-23_Handsoldering" H 9400 5750 50  0001 C CNN
 F 3 "" H 9200 5650 50  0000 C CNN
 	1    9200 5650
@@
 Text Label 8200 5650 0    60   ~ 0
 PB15
+$Comp
+L R R7
+U 1 1 5857A47C
+P 3250 6550
+F 0 "R7" V 3330 6550 50  0000 C CNN
+F 1 "0" V 3250 6550 50  0000 C CNN
+F 2 "Resistors_SMD:R_0805_HandSoldering" V 3180 6550 50  0001 C CNN
+F 3 "" H 3250 6550 50  0000 C CNN
+	1    3250 6550
+	0    1    1    0
+$EndComp
+Wire Wire Line
+	3400 6550 3400 6400
+Wire Wire Line
+	3400 6550 3700 6550
+Wire Wire Line
+	3700 6550 3700 6400
 $EndSCHEMATC

Commit message: Initial layout
Parts:
- removed W1: TEST_VDD, Measurement_Points:Measurement_Point_Round-SMD-Pad_Big, symbol TEST_1P
- added P2: PWR, Pin_Headers:Pin_Header_Straight_1x02, symbol CONN_01X02
- L1: footprint Inductors:Inductor_1212 -> Inductors:Inductor_Taiyo-Yuden_NR-30xx_HandSoldering
Connections:
- wire segments 82 -> 81
Changed lines of the file:
@@
 F 0 "L1" V 1350 6550 50  0000 C CNN
 F 1 "INDUCTOR" V 1500 6550 50  0000 C CNN
-F 2 "Inductors:Inductor_1212" H 1400 6550 50  0001 C CNN
+F 2 "Inductors:Inductor_Taiyo-Yuden_NR-30xx_HandSoldering" H 1400 6550 50  0001 C CNN
 F 3 "" H 1400 6550 50  0000 C CNN
 	1    1400 6550
@@
 $EndComp
 $Comp
-L TEST_1P W1
-U 1 1 58557FAC
-P 3400 6400
-F 0 "W1" H 3400 6670 50  0000 C CNN
-F 1 "TEST_VDD" H 3400 6600 50  0000 C CNN
-F 2 "Measurement_Points:Measurement_Point_Round-SMD-Pad_Big" H 3600 6400 50  0001 C CNN
-F 3 "" H 3600 6400 50  0000 C CNN
-	1    3400 6400
-	1    0    0    -1
-$EndComp
-$Comp
 L Q_NMOS_GSD Q1
 U 1 1 585590EB
@@
 $EndComp
 Wire Wire Line
-	3400 6550 3400 6400
-Wire Wire Line
 	3400 6550 3700 6550
 Wire Wire Line
 	3700 6550 3700 6400
+$Comp
+L CONN_01X02 P2
+U 1 1 5857BC53
+P 950 5700
+F 0 "P2" H 950 5850 50  0000 C CNN
+F 1 "PWR" V 1050 5700 50  0000 C CNN
+F 2 "Pin_Headers:Pin_Header_Straight_1x02" H 950 5700 50  0001 C CNN
+F 3 "" H 950 5700 50  0000 C CNN
+	1    950  5700
+	-1   0    0    -1
+$EndComp
+$Comp
+L +BATT #PWR028
+U 1 1 5857BD0C
+P 1150 5650
+F 0 "#PWR028" H 1150 5500 50  0001 C CNN
+F 1 "+BATT" H 1150 5790 50  0000 C CNN
+F 2 "" H 1150 5650 50  0000 C CNN
+F 3 "" H 1150 5650 50  0000 C CNN
+	1    1150 5650
+	1    0    0    -1
+$EndComp
+$Comp
+L Earth #PWR029
+U 1 1 5857BE4D
+P 1150 5750
+F 0 "#PWR029" H 1150 5500 50  0001 C CNN
+F 1 "Earth" H 1150 5600 50  0001 C CNN
+F 2 "" H 1150 5750 50  0000 C CNN
+F 3 "" H 1150 5750 50  0000 C CNN
+	1    1150 5750
+	1    0    0    -1
+$EndComp
 $EndSCHEMATC

Commit message: Layout to fit the enclosure
Parts:
- removed D1: LED, LEDs:LED_0805, symbol LED
- removed R1: 820, Resistors_SMD:R_0805_HandSoldering, symbol R
Connections:
- wire segments 81 -> 78
Changed lines of the file:
@@
 	1    0    0    -1
 $EndComp
-$Comp
-L LED D1
-U 1 1 58076AE7
-P 9300 2200
-F 0 "D1" H 9300 2300 50  0000 C CNN
-F 1 "LED" H 9300 2100 50  0000 C CNN
-F 2 "LEDs:LED_0805" H 9300 2200 50  0001 C CNN
-F 3 "" H 9300 2200 50  0000 C CNN
-	1    9300 2200
-	-1   0    0    -1
-$EndComp
-$Comp
-L R R1
-U 1 1 580770D7
-P 8950 2200
-F 0 "R1" V 9030 2200 50  0000 C CNN
-F 1 "820" V 8950 2200 50  0000 C CNN
-F 2 "Resistors_SMD:R_0805_HandSoldering" V 8880 2200 50  0001 C CNN
-F 3 "" H 8950 2200 50  0000 C CNN
-	1    8950 2200
-	0    -1   1    0
-$EndComp
-$Comp
-L Earth #PWR014
-U 1 1 58077163
-P 9600 2300
-F 0 "#PWR014" H 9600 2050 50  0001 C CNN
-F 1 "Earth" H 9600 2150 50  0001 C CNN
-F 2 "" H 9600 2300 50  0000 C CNN
-F 3 "" H 9600 2300 50  0000 C CNN
-	1    9600 2300
-	-1   0    0    -1
-$EndComp
-Wire Wire Line
-	9600 2300 9600 2200
-Wire Wire Line
-	9600 2200 9500 2200
-Wire Wire Line
-	8600 2200 8800 2200
 Wire Wire Line
 	5200 1750 5200 2000
@@
 Connection ~ 3600 5700
 NoConn ~ 4600 4700
-Text GLabel 8600 2200 0    60   Input ~ 0
-PA5
 Text Label 8500 3350 0    60   ~ 0
 LCD_COM0

Commit message: HAL_PWR_EnterSTANDBYMode()
Connections:
- net BUTTON1 is gone; now on net BUTTON0: C10.1, R4.1, U1.41 (PB5)
- net BUTTON2 is gone; now on net BUTTON0: C11.1, R5.1, U1.42 (PB6)
- net BUTTON0: now also U1.10 (PAO)
- no-connect marks 16 -> 15
Changed lines of the file:
@@
 NoConn ~ 6550 3600
 NoConn ~ 6550 3700
-NoConn ~ 4600 2300
 NoConn ~ 4600 2700
 NoConn ~ 4600 3400
@@
 	1    0    0    -1
 $EndComp
+Text Label 3900 2300 0    60   ~ 0
+WAKEUP_PIN1
+Wire Wire Line
+	3500 2300 4600 2300
+Text Label 3500 1900 2    60   ~ 0
+BUTTON0
+Text Label 3500 2100 2    60   ~ 0
+BUTTON1
+Text Label 3500 2300 2    60   ~ 0
+BUTTON2
+Wire Wire Line
+	3900 1900 3900 2300
+Connection ~ 3900 2100
+Wire Wire Line
+	3500 1900 3900 1900
+Wire Wire Line
+	3500 2100 3900 2100
+Connection ~ 3900 2300
 $EndSCHEMATC
