File: kicad/stm32l053c.sch (KiCad schematic (older format))
At the start: 35 parts, among them P1 SWD, P2 PWR, Q1 Q_PNP_BEC, SW1 SW_PUSH, SW2 SW_PUSH, SW3 SW_PUSH, U1 STM32L053C8_LQFP48, U2 TLV61225, U3 um66t, Y1 Crystal

Commit message: Moved the melody pin
Parts:
- R6: value 1K -> 220
Connections:
- wire segments 92 -> 93
- no-connect marks 14 -> 13
Changed lines of the file:
@@
 NoConn ~ 6550 3100
 NoConn ~ 6550 3300
-NoConn ~ 6550 3500
 NoConn ~ 6550 3600
 NoConn ~ 6550 3700
@@
 P 8350 3650
 F 0 "R6" V 8430 3650 50  0000 C CNN
-F 1 "1K" V 8350 3650 50  0000 C CNN
+F 1 "220" V 8350 3650 50  0000 C CNN
 F 2 "Resistors_SMD:R_0805_HandSoldering" V 8280 3650 50  0001 C CNN
 F 3 "" H 8350 3650 50  0000 C CNN
@@
 	1    0    0    -1
 $EndComp
-Text Label 7100 3800 2    60   ~ 0
+Text Label 7100 3500 2    60   ~ 0
 MELODY
 Wire Wire Line
@@
 Wire Wire Line
 	6550 3400 7250 3400
-Wire Wire Line
-	6550 3800 7100 3800
 $Comp
 L R R1
@@
 	1    0    0    -1
 $EndComp
+Wire Wire Line
+	6550 3500 7100 3500
+Wire Wire Line
+	7100 3500 7100 3800
 $EndSCHEMATC

Commit message: Fixed the melody output
Parts:
- added R8: 1K, Resistors_SMD:R_0805_HandSoldering, symbol R
Connections:
- wire segments 93 -> 92
Changed lines of the file:
@@
 $EndDescr
 $Comp
-L Earth #PWR01
+L Earth #PWR28
 U 1 1 58021BE1
 P 4900 7200
-F 0 "#PWR01" H 4900 6950 50  0001 C CNN
+F 0 "#PWR28" H 4900 6950 50  0001 C CNN
 F 1 "Earth" H 4900 7050 50  0001 C CNN
 F 2 "" H 4900 7200 50  0000 C CNN
@@
 $EndComp
 $Comp
-L VDD #PWR02
+L VDD #PWR26
 U 1 1 58021C2A
 P 4900 6900
-F 0 "#PWR02" H 4900 6750 50  0001 C CNN
+F 0 "#PWR26" H 4900 6750 50  0001 C CNN
 F 1 "VDD" H 4900 7050 50  0000 C CNN
 F 2 "" H 4900 6900 50  0000 C CNN
@@
 $EndComp
 $Comp
-L GNDA #PWR03
+L GNDA #PWR20
 U 1 1 58021F75
 P 5100 6300
-F 0 "#PWR03" H 5100 6050 50  0001 C CNN
+F 0 "#PWR20" H 5100 6050 50  0001 C CNN
 F 1 "GNDA" H 5100 6150 50  0000 C CNN
 F 2 "" H 5100 6300 50  0000 C CNN
@@
 $EndComp
 $Comp
-L Earth #PWR04
+L Earth #PWR21
 U 1 1 58021F89
 P 5600 6300
-F 0 "#PWR04" H 5600 6050 50  0001 C CNN
+F 0 "#PWR21" H 5600 6050 50  0001 C CNN
 F 1 "Earth" H 5600 6150 50  0001 C CNN
 F 2 "" H 5600 6300 50  0000 C CNN
@@
 $EndComp
 $Comp
-L GNDA #PWR05
+L GNDA #PWR18
 U 1 1 58022154
 P 5150 5800
-F 0 "#PWR05" H 5150 5550 50  0001 C CNN
+F 0 "#PWR18" H 5150 5550 50  0001 C CNN
 F 1 "GNDA" H 5150 5650 50  0000 C CNN
 F 2 "" H 5150 5800 50  0000 C CNN
@@
 $EndComp
 $Comp
-L Earth #PWR06
+L Earth #PWR19
 U 1 1 580221FA
 P 5650 5800
-F 0 "#PWR06" H 5650 5550 50  0001 C CNN
+F 0 "#PWR19" H 5650 5550 50  0001 C CNN
 F 1 "Earth" H 5650 5650 50  0001 C CNN
 F 2 "" H 5650 5800 50  0000 C CNN
@@
 $EndComp
 $Comp
-L VDD #PWR07
+L VDD #PWR1
 U 1 1 5802295B
 P 5450 1050
-F 0 "#PWR07" H 5450 900 50  0001 C CNN
+F 0 "#PWR1" H 5450 900 50  0001 C CNN
 F 1 "VDD" H 5450 1200 50  0000 C CNN
 F 2 "" H 5450 1050 50  0000 C CNN
@@
 $EndComp
 $Comp
-L Earth #PWR08
+L Earth #PWR4
 U 1 1 5803310F
 P 4800 1800
-F 0 "#PWR08" H 4800 1550 50  0001 C CNN
+F 0 "#PWR4" H 4800 1550 50  0001 C CNN
 F 1 "Earth" H 4800 1650 50  0001 C CNN
 F 2 "" H 4800 1800 50  0000 C CNN
@@
 $EndComp
 $Comp
-L Earth #PWR09
+L Earth #PWR3
 U 1 1 580369A9
 P 2150 1400
-F 0 "#PWR09" H 2150 1150 50  0001 C CNN
+F 0 "#PWR3" H 2150 1150 50  0001 C CNN
 F 1 "Earth" H 2150 1250 50  0001 C CNN
 F 2 "" H 2150 1400 50  0000 C CNN
@@
 NRST
 $Comp
-L VDD #PWR010
+L VDD #PWR2
 U 1 1 5803734F
 P 1650 1200
-F 0 "#PWR010" H 1650 1050 50  0001 C CNN
+F 0 "#PWR2" H 1650 1050 50  0001 C CNN
 F 1 "VDD" H 1650 1350 50  0000 C CNN
 F 2 "" H 1650 1200 50  0000 C CNN
@@
 $EndComp
 $Comp
-L Earth #PWR011
+L Earth #PWR29
 U 1 1 5803BDC8
 P 5950 7200
-F 0 "#PWR011" H 5950 6950 50  0001 C CNN
+F 0 "#PWR29" H 5950 6950 50  0001 C CNN
 F 1 "Earth" H 5950 7050 50  0001 C CNN
 F 2 "" H 5950 7200 50  0000 C CNN
@@
 $EndComp
 $Comp
-L Earth #PWR012
+L Earth #PWR14
 U 1 1 58065816
 P 6550 5400
-F 0 "#PWR012" H 6550 5150 50  0001 C CNN
+F 0 "#PWR14" H 6550 5150 50  0001 C CNN
 F 1 "Earth" H 6550 5250 50  0001 C CNN
 F 2 "" H 6550 5400 50  0000 C CNN
@@
 $EndComp
 $Comp
-L Earth #PWR013
+L Earth #PWR16
 U 1 1 5806680D
 P 3600 5700
-F 0 "#PWR013" H 3600 5450 50  0001 C CNN
+F 0 "#PWR16" H 3600 5450 50  0001 C CNN
 F 1 "Earth" H 3600 5550 50  0001 C CNN
 F 2 "" H 3600 5700 50  0000 C CNN
@@
 $EndComp
 $Comp
-L +BATT #PWR014
+L +BATT #PWR23
 U 1 1 584F2368
 P 850 6750
-F 0 "#PWR014" H 850 6600 50  0001 C CNN
+F 0 "#PWR23" H 850 6600 50  0001 C CNN
 F 1 "+BATT" H 850 6890 50  0000 C CNN
 F 2 "" H 850 6750 50  0000 C CNN
@@
 $EndComp
 $Comp
-L Earth #PWR015
+L Earth #PWR25
 U 1 1 584F287E
 P 2850 6850
-F 0 "#PWR015" H 2850 6600 50  0001 C CNN
+F 0 "#PWR25" H 2850 6600 50  0001 C CNN
 F 1 "Earth" H 2850 6700 50  0001 C CNN
 F 2 "" H 2850 6850 50  0000 C CNN
@@
 $EndComp
 $Comp
-L Earth #PWR016
+L Earth #PWR24
 U 1 1 584F28E3
 P 1700 6850
-F 0 "#PWR016" H 1700 6600 50  0001 C CNN
+F 0 "#PWR24" H 1700 6600 50  0001 C CNN
 F 1 "Earth" H 1700 6700 50  0001 C CNN
 F 2 "" H 1700 6850 50  0000 C CNN
@@
 $EndComp
 $Comp
-L Earth #PWR017
+L Earth #PWR27
 U 1 1 584F2924
 P 1250 7050
-F 0 "#PWR017" H 1250 6800 50  0001 C CNN
+F 0 "#PWR27" H 1250 6800 50  0001 C CNN
 F 1 "Earth" H 1250 6900 50  0001 C CNN
 F 2 "" H 1250 7050 50  0000 C CNN
@@
 $EndComp
 $Comp
-L VDD #PWR018
+L VDD #PWR22
 U 1 1 584F2A51
 P 3700 6400
-F 0 "#PWR018" H 3700 6250 50  0001 C CNN
+F 0 "#PWR22" H 3700 6250 50  0001 C CNN
 F 1 "VDD" H 3700 6550 50  0000 C CNN
 F 2 "" H 3700 6400 50  0000 C CNN
@@
 $EndComp
 $Comp
-L VDD #PWR019
+L VDD #PWR6
 U 1 1 585069C3
 P 1300 2700
-F 0 "#PWR019" H 1300 2550 50  0001 C CNN
+F 0 "#PWR6" H 1300 2550 50  0001 C CNN
 F 1 "VDD" H 1300 2850 50  0000 C CNN
 F 2 "" H 1300 2700 50  0000 C CNN
@@
 $EndComp
 $Comp
-L VDD #PWR020
+L VDD #PWR8
 U 1 1 58506BE4
 P 1300 3300
-F 0 "#PWR020" H 1300 3150 50  0001 C CNN
+F 0 "#PWR8" H 1300 3150 50  0001 C CNN
 F 1 "VDD" H 1300 3450 50  0000 C CNN
 F 2 "" H 1300 3300 50  0000 C CNN
@@
 $EndComp
 $Comp
-L VDD #PWR021
+L VDD #PWR11
 U 1 1 58506C86
 P 1300 3900
-F 0 "#PWR021" H 1300 3750 50  0001 C CNN
+F 0 "#PWR11" H 1300 3750 50  0001 C CNN
 F 1 "VDD" H 1300 4050 50  0000 C CNN
 F 2 "" H 1300 3900 50  0000 C CNN
@@
 $EndComp
 $Comp
-L Earth #PWR022
+L Earth #PWR7
 U 1 1 5851A35F
 P 2450 3150
-F 0 "#PWR022" H 2450 2900 50  0001 C CNN
+F 0 "#PWR7" H 2450 2900 50  0001 C CNN
 F 1 "Earth" H 2450 3000 50  0001 C CNN
 F 2 "" H 2450 3150 50  0000 C CNN
@@
 $EndComp
 $Comp
-L Earth #PWR023
+L Earth #PWR9
 U 1 1 5851A4F4
 P 2450 3750
-F 0 "#PWR023" H 2450 3500 50  0001 C CNN
+F 0 "#PWR9" H 2450 3500 50  0001 C CNN
 F 1 "Earth" H 2450 3600 50  0001 C CNN
 F 2 "" H 2450 3750 50  0000 C CNN
@@
 $EndComp
 $Comp
-L Earth #PWR024
+L Earth #PWR13
 U 1 1 5851A54D
 P 2450 4350
-F 0 "#PWR024" H 2450 4100 50  0001 C CNN
+F 0 "#PWR13" H 2450 4100 50  0001 C CNN
 F 1 "Earth" H 2450 4200 50  0001 C CNN
 F 2 "" H 2450 4350 50  0000 C CNN
@@
 $EndComp
 $Comp
-L Earth #PWR025
+L Earth #PWR10
 U 1 1 5851B22D
 P 8900 3850
-F 0 "#PWR025" H 8900 3600 50  0001 C CNN
+F 0 "#PWR10" H 8900 3600 50  0001 C CNN
 F 1 "Earth" H 8900 3700 50  0001 C CNN
 F 2 "" H 8900 3850 50  0000 C CNN
@@
 $EndComp
 $Comp
-L +BATT #PWR027
+L +BATT #PWR15
 U 1 1 5857BD0C
 P 1150 5650
-F 0 "#PWR027" H 1150 5500 50  0001 C CNN
+F 0 "#PWR15" H 1150 5500 50  0001 C CNN
 F 1 "+BATT" H 1150 5790 50  0000 C CNN
 F 2 "" H 1150 5650 50  0000 C CNN
@@
 $EndComp
 $Comp
-L Earth #PWR028
+L Earth #PWR17
 U 1 1 5857BE4D
 P 1150 5750
-F 0 "#PWR028" H 1150 5500 50  0001 C CNN
+F 0 "#PWR17" H 1150 5500 50  0001 C CNN
 F 1 "Earth" H 1150 5600 50  0001 C CNN
 F 2 "" H 1150 5750 50  0000 C CNN
@@
 $EndComp
 $Comp
-L Earth #PWR029
+L Earth #PWR12
 U 1 1 586A57FA
 P 7100 3900
-F 0 "#PWR029" H 7100 3650 50  0001 C CNN
+F 0 "#PWR12" H 7100 3650 50  0001 C CNN
 F 1 "Earth" H 7100 3750 50  0001 C CNN
 F 2 "" H 7100 3900 50  0000 C CNN
@@
 Connection ~ 8900 3100
 $Comp
-L +BATT #PWR?
+L +BATT #PWR5
 U 1 1 586A907B
 P 8900 2650
-F 0 "#PWR?" H 8900 2500 50  0001 C CNN
+F 0 "#PWR5" H 8900 2500 50  0001 C CNN
 F 1 "+BATT" H 8900 2790 50  0000 C CNN
 F 2 "" H 8900 2650 50  0000 C CNN
@@
 Wire Wire Line
 	6550 3500 7100 3500
-Wire Wire Line
-	7100 3500 7100 3800
+$Comp
+L R R8
+U 1 1 586AB55A
+P 7100 3650
+F 0 "R8" V 7180 3650 50  0000 C CNN
+F 1 "1K" V 7100 3650 50  0000 C CNN
+F 2 "Resistors_SMD:R_0805_HandSoldering" V 7030 3650 50  0001 C CNN
+F 3 "" H 7100 3650 50  0000 C CNN
+	1    7100 3650
+	-1   0    0    1
+$EndComp
 $EndSCHEMATC

Commit message: Stop noise on the buzzer
Parts:
- R8: value 1K -> 10K
Connections:
- wire segments 92 -> 94
Other:
- moved on the sheet: R8
Changed lines of the file:
@@
 $EndDescr
 $Comp
-L Earth #PWR28
+L Earth #PWR01
 U 1 1 58021BE1
 P 4900 7200
-F 0 "#PWR28" H 4900 6950 50  0001 C CNN
+F 0 "#PWR01" H 4900 6950 50  0001 C CNN
 F 1 "Earth" H 4900 7050 50  0001 C CNN
 F 2 "" H 4900 7200 50  0000 C CNN
@@
 $EndComp
 $Comp
-L VDD #PWR26
+L VDD #PWR02
 U 1 1 58021C2A
 P 4900 6900
-F 0 "#PWR26" H 4900 6750 50  0001 C CNN
+F 0 "#PWR02" H 4900 6750 50  0001 C CNN
 F 1 "VDD" H 4900 7050 50  0000 C CNN
 F 2 "" H 4900 6900 50  0000 C CNN
@@
 $EndComp
 $Comp
-L GNDA #PWR20
+L GNDA #PWR03
 U 1 1 58021F75
 P 5100 6300
-F 0 "#PWR20" H 5100 6050 50  0001 C CNN
+F 0 "#PWR03" H 5100 6050 50  0001 C CNN
 F 1 "GNDA" H 5100 6150 50  0000 C CNN
 F 2 "" H 5100 6300 50  0000 C CNN
@@
 $EndComp
 $Comp
-L Earth #PWR21
+L Earth #PWR04
 U 1 1 58021F89
 P 5600 6300
-F 0 "#PWR21" H 5600 6050 50  0001 C CNN
+F 0 "#PWR04" H 5600 6050 50  0001 C CNN
 F 1 "Earth" H 5600 6150 50  0001 C CNN
 F 2 "" H 5600 6300 50  0000 C CNN
@@
 $EndComp
 $Comp
-L GNDA #PWR18
+L GNDA #PWR05
 U 1 1 58022154
 P 5150 5800
-F 0 "#PWR18" H 5150 5550 50  0001 C CNN
+F 0 "#PWR05" H 5150 5550 50  0001 C CNN
 F 1 "GNDA" H 5150 5650 50  0000 C CNN
 F 2 "" H 5150 5800 50  0000 C CNN
@@
 $EndComp
 $Comp
-L Earth #PWR19
+L Earth #PWR06
 U 1 1 580221FA
 P 5650 5800
-F 0 "#PWR19" H 5650 5550 50  0001 C CNN
+F 0 "#PWR06" H 5650 5550 50  0001 C CNN
 F 1 "Earth" H 5650 5650 50  0001 C CNN
 F 2 "" H 5650 5800 50  0000 C CNN
@@
 $EndComp
 $Comp
-L VDD #PWR1
+L VDD #PWR07
 U 1 1 5802295B
 P 5450 1050
-F 0 "#PWR1" H 5450 900 50  0001 C CNN
+F 0 "#PWR07" H 5450 900 50  0001 C CNN
 F 1 "VDD" H 5450 1200 50  0000 C CNN
 F 2 "" H 5450 1050 50  0000 C CNN
@@
 $EndComp
 $Comp
-L Earth #PWR4
+L Earth #PWR08
 U 1 1 5803310F
 P 4800 1800
-F 0 "#PWR4" H 4800 1550 50  0001 C CNN
+F 0 "#PWR08" H 4800 1550 50  0001 C CNN
 F 1 "Earth" H 4800 1650 50  0001 C CNN
 F 2 "" H 4800 1800 50  0000 C CNN
@@
 $EndComp
 $Comp
-L Earth #PWR3
+L Earth #PWR09
 U 1 1 580369A9
 P 2150 1400
-F 0 "#PWR3" H 2150 1150 50  0001 C CNN
+F 0 "#PWR09" H 2150 1150 50  0001 C CNN
 F 1 "Earth" H 2150 1250 50  0001 C CNN
 F 2 "" H 2150 1400 50  0000 C CNN
@@
 NRST
 $Comp
-L VDD #PWR2
+L VDD #PWR010
 U 1 1 5803734F
 P 1650 1200
-F 0 "#PWR2" H 1650 1050 50  0001 C CNN
+F 0 "#PWR010" H 1650 1050 50  0001 C CNN
 F 1 "VDD" H 1650 1350 50  0000 C CNN
 F 2 "" H 1650 1200 50  0000 C CNN
@@
 $EndComp
 $Comp
-L Earth #PWR29
+L Earth #PWR011
 U 1 1 5803BDC8
 P 5950 7200
-F 0 "#PWR29" H 5950 6950 50  0001 C CNN
+F 0 "#PWR011" H 5950 6950 50  0001 C CNN
 F 1 "Earth" H 5950 7050 50  0001 C CNN
 F 2 "" H 5950 7200 50  0000 C CNN
@@
 $EndComp
 $Comp
-L Earth #PWR14
+L Earth #PWR012
 U 1 1 58065816
 P 6550 5400
-F 0 "#PWR14" H 6550 5150 50  0001 C CNN
+F 0 "#PWR012" H 6550 5150 50  0001 C CNN
 F 1 "Earth" H 6550 5250 50  0001 C CNN
 F 2 "" H 6550 5400 50  0000 C CNN
@@
 $EndComp
 $Comp
-L Earth #PWR16
+L Earth #PWR013
 U 1 1 5806680D
 P 3600 5700
-F 0 "#PWR16" H 3600 5450 50  0001 C CNN
+F 0 "#PWR013" H 3600 5450 50  0001 C CNN
 F 1 "Earth" H 3600 5550 50  0001 C CNN
 F 2 "" H 3600 5700 50  0000 C CNN
@@
 $EndComp
 $Comp
-L +BATT #PWR23
+L +BATT #PWR014
 U 1 1 584F2368
 P 850 6750
-F 0 "#PWR23" H 850 6600 50  0001 C CNN
+F 0 "#PWR014" H 850 6600 50  0001 C CNN
 F 1 "+BATT" H 850 6890 50  0000 C CNN
 F 2 "" H 850 6750 50  0000 C CNN
@@
 $EndComp
 $Comp
-L Earth #PWR25
+L Earth #PWR015
 U 1 1 584F287E
 P 2850 6850
-F 0 "#PWR25" H 2850 6600 50  0001 C CNN
+F 0 "#PWR015" H 2850 6600 50  0001 C CNN
 F 1 "Earth" H 2850 6700 50  0001 C CNN
 F 2 "" H 2850 6850 50  0000 C CNN
@@
 $EndComp
 $Comp
-L Earth #PWR24
+L Earth #PWR016
 U 1 1 584F28E3
 P 1700 6850
-F 0 "#PWR24" H 1700 6600 50  0001 C CNN
+F 0 "#PWR016" H 1700 6600 50  0001 C CNN
 F 1 "Earth" H 1700 6700 50  0001 C CNN
 F 2 "" H 1700 6850 50  0000 C CNN
@@
 $EndComp
 $Comp
-L Earth #PWR27
+L Earth #PWR017
 U 1 1 584F2924
 P 1250 7050
-F 0 "#PWR27" H 1250 6800 50  0001 C CNN
+F 0 "#PWR017" H 1250 6800 50  0001 C CNN
 F 1 "Earth" H 1250 6900 50  0001 C CNN
 F 2 "" H 1250 7050 50  0000 C CNN
@@
 $EndComp
 $Comp
-L VDD #PWR22
+L VDD #PWR018
 U 1 1 584F2A51
 P 3700 6400
-F 0 "#PWR22" H 3700 6250 50  0001 C CNN
+F 0 "#PWR018" H 3700 6250 50  0001 C CNN
 F 1 "VDD" H 3700 6550 50  0000 C CNN
 F 2 "" H 3700 6400 50  0000 C CNN
@@
 $EndComp
 $Comp
-L VDD #PWR6
+L VDD #PWR019
 U 1 1 585069C3
 P 1300 2700
-F 0 "#PWR6" H 1300 2550 50  0001 C CNN
+F 0 "#PWR019" H 1300 2550 50  0001 C CNN
 F 1 "VDD" H 1300 2850 50  0000 C CNN
 F 2 "" H 1300 2700 50  0000 C CNN
@@
 $EndComp
 $Comp
-L VDD #PWR8
+L VDD #PWR020
 U 1 1 58506BE4
 P 1300 3300
-F 0 "#PWR8" H 1300 3150 50  0001 C CNN
+F 0 "#PWR020" H 1300 3150 50  0001 C CNN
 F 1 "VDD" H 1300 3450 50  0000 C CNN
 F 2 "" H 1300 3300 50  0000 C CNN
@@
 $EndComp
 $Comp
-L VDD #PWR11
+L VDD #PWR021
 U 1 1 58506C86
 P 1300 3900
-F 0 "#PWR11" H 1300 3750 50  0001 C CNN
+F 0 "#PWR021" H 1300 3750 50  0001 C CNN
 F 1 "VDD" H 1300 4050 50  0000 C CNN
 F 2 "" H 1300 3900 50  0000 C CNN
@@
 $EndComp
 $Comp
-L Earth #PWR7
+L Earth #PWR022
 U 1 1 5851A35F
 P 2450 3150
-F 0 "#PWR7" H 2450 2900 50  0001 C CNN
+F 0 "#PWR022" H 2450 2900 50  0001 C CNN
 F 1 "Earth" H 2450 3000 50  0001 C CNN
 F 2 "" H 2450 3150 50  0000 C CNN
@@
 $EndComp
 $Comp
-L Earth #PWR9
+L Earth #PWR023
 U 1 1 5851A4F4
 P 2450 3750
-F 0 "#PWR9" H 2450 3500 50  0001 C CNN
+F 0 "#PWR023" H 2450 3500 50  0001 C CNN
 F 1 "Earth" H 2450 3600 50  0001 C CNN
 F 2 "" H 2450 3750 50  0000 C CNN
@@
 $EndComp
 $Comp
-L Earth #PWR13
+L Earth #PWR024
 U 1 1 5851A54D
 P 2450 4350
-F 0 "#PWR13" H 2450 4100 50  0001 C CNN
+F 0 "#PWR024" H 2450 4100 50  0001 C CNN
 F 1 "Earth" H 2450 4200 50  0001 C CNN
 F 2 "" H 2450 4350 50  0000 C CNN
@@
 $EndComp
 $Comp
-L Earth #PWR10
+L Earth #PWR025
 U 1 1 5851B22D
 P 8900 3850
-F 0 "#PWR10" H 8900 3600 50  0001 C CNN
+F 0 "#PWR025" H 8900 3600 50  0001 C CNN
 F 1 "Earth" H 8900 3700 50  0001 C CNN
 F 2 "" H 8900 3850 50  0000 C CNN
@@
 $EndComp
 $Comp
-L +BATT #PWR15
+L +BATT #PWR026
 U 1 1 5857BD0C
 P 1150 5650
-F 0 "#PWR15" H 1150 5500 50  0001 C CNN
+F 0 "#PWR026" H 1150 5500 50  0001 C CNN
 F 1 "+BATT" H 1150 5790 50  0000 C CNN
 F 2 "" H 1150 5650 50  0000 C CNN
@@
 $EndComp
 $Comp
-L Earth #PWR17
+L Earth #PWR027
 U 1 1 5857BE4D
 P 1150 5750
-F 0 "#PWR17" H 1150 5500 50  0001 C CNN
+F 0 "#PWR027" H 1150 5500 50  0001 C CNN
 F 1 "Earth" H 1150 5600 50  0001 C CNN
 F 2 "" H 1150 5750 50  0000 C CNN
@@
 $EndComp
 $Comp
-L Earth #PWR12
+L Earth #PWR028
 U 1 1 586A57FA
 P 7100 3900
-F 0 "#PWR12" H 7100 3650 50  0001 C CNN
+F 0 "#PWR028" H 7100 3650 50  0001 C CNN
 F 1 "Earth" H 7100 3750 50  0001 C CNN
 F 2 "" H 7100 3900 50  0000 C CNN
@@
 Connection ~ 8900 3100
 $Comp
-L +BATT #PWR5
+L +BATT #PWR029
 U 1 1 586A907B
 P 8900 2650
-F 0 "#PWR5" H 8900 2500 50  0001 C CNN
+F 0 "#PWR029" H 8900 2500 50  0001 C CNN
 F 1 "+BATT" H 8900 2790 50  0000 C CNN
 F 2 "" H 8900 2650 50  0000 C CNN
@@
 L R R8
 U 1 1 586AB55A
-P 7100 3650
-F 0 "R8" V 7180 3650 50  0000 C CNN
-F 1 "1K" V 7100 3650 50  0000 C CNN
-F 2 "Resistors_SMD:R_0805_HandSoldering" V 7030 3650 50  0001 C CNN
-F 3 "" H 7100 3650 50  0000 C CNN
-	1    7100 3650
+P 8100 3900
+F 0 "R8" V 8180 3900 50  0000 C CNN
+F 1 "10K" V 8100 3900 50  0000 C CNN
+F 2 "Resistors_SMD:R_0805_HandSoldering" V 8030 3900 50  0001 C CNN
+F 3 "" H 8100 3900 50  0000 C CNN
+	1    8100 3900
 	-1   0    0    1
 $EndComp
+Wire Wire Line
+	7100 3500 7100 3800
+$Comp
+L Earth #PWR?
+U 1 1 586AC8CF
+P 8100 4050
+F 0 "#PWR?" H 8100 3800 50  0001 C CNN
+F 1 "Earth" H 8100 3900 50  0001 C CNN
+F 2 "" H 8100 4050 50  0000 C CNN
+F 3 "" H 8100 4050 50  0000 C CNN
+	1    8100 4050
+	1    0    0    -1
+$EndComp
+Wire Wire Line
+	8100 3750 8100 3650
+Connection ~ 8100 3650
 $EndSCHEMATC

Commit message: Pull down on the buzzer transistor
Connections:
- wire segments 94 -> 112
Changed lines of the file:
@@
 Connection ~ 5450 5650
 Wire Wire Line
-	5450 1050 5450 2000
+	5450 1050 5450 1250
+Wire Wire Line
+	5450 1250 5450 2000
 Wire Wire Line
 	5550 1250 5550 2000
@@
 	5300 1250 5300 2000
 Wire Wire Line
-	5300 1250 5900 1250
+	5300 1250 5450 1250
+Wire Wire Line
+	5450 1250 5550 1250
+Wire Wire Line
+	5550 1250 5900 1250
 Connection ~ 5450 1250
 Wire Wire Line
@@
 	6550 2600 7100 2600
 Wire Wire Line
-	5450 5650 5650 5650
+	5450 5650 5550 5650
+Wire Wire Line
+	5550 5650 5650 5650
 Wire Wire Line
 	3450 4800 4600 4800
 Wire Wire Line
-	3450 4800 3450 5250
+	3450 4800 3450 5050
+Wire Wire Line
+	3450 5050 3450 5250
 Connection ~ 3450 5050
 Wire Wire Line
 	3750 4900 4600 4900
 Wire Wire Line
-	3750 4900 3750 5250
+	3750 4900 3750 5050
+Wire Wire Line
+	3750 5050 3750 5250
 Connection ~ 3750 5050
 Wire Wire Line
 	3750 5700 3750 5550
 Wire Wire Line
-	3450 5700 3750 5700
+	3450 5700 3600 5700
+Wire Wire Line
+	3600 5700 3750 5700
 Wire Wire Line
 	3450 5550 3450 5700
 Connection ~ 3600 5700
 Wire Wire Line
-	850  6750 1700 6750
+	850  6750 1100 6750
+Wire Wire Line
+	1100 6750 1250 6750
+Wire Wire Line
+	1250 6750 1600 6750
+Wire Wire Line
+	1600 6750 1700 6750
 Connection ~ 1250 6750
 Wire Wire Line
@@
 Connection ~ 1600 6750
 Wire Wire Line
-	2600 6550 3100 6550
+	2600 6550 2700 6550
+Wire Wire Line
+	2700 6550 2850 6550
+Wire Wire Line
+	2850 6550 3100 6550
 Connection ~ 2850 6550
 Wire Wire Line
@@
 	2450 2850 3000 2850
 Wire Wire Line
-	8900 3000 8900 3450
+	8900 3000 8900 3100
+Wire Wire Line
+	8900 3100 8900 3450
 Wire Wire Line
 	8600 3650 8500 3650
 Wire Wire Line
-	8200 3650 7800 3650
+	8200 3650 8100 3650
+Wire Wire Line
+	8100 3650 7700 3650
 Wire Wire Line
 	3400 6550 3700 6550
@@
 $EndComp
 Wire Wire Line
-	7550 3400 7800 3400
+	7550 3400 7700 3400
 $Comp
 L D_Schottky D3
@@
 	2600 1700 3200 1700
 Wire Wire Line
-	3500 2300 4600 2300
+	3500 2300 3800 2300
+Wire Wire Line
+	3800 2300 4600 2300
 Wire Wire Line
 	3500 1700 3800 1700
 Wire Wire Line
-	3800 1700 3800 2300
+	3800 1700 3800 2000
+Wire Wire Line
+	3800 2000 3800 2300
 Wire Wire Line
 	3500 2000 3800 2000
@@
 $EndComp
 Wire Wire Line
-	7800 4000 7700 4000
-Wire Wire Line
-	7800 3400 7800 4000
-Connection ~ 7800 3650
+	7700 4000 7700 4000
+Wire Wire Line
+	7700 3400 7700 3650
+Wire Wire Line
+	7700 3650 7700 4000
+Connection ~ 7700 3650
 Text Notes 6750 4350 0    60   ~ 0
 Either BUZZER or MELODY
@@
 $EndComp
 Wire Wire Line
-	8900 2900 8900 2650
+	8900 2900 8900 2800
+Wire Wire Line
+	8900 2800 8900 2650
 Wire Wire Line
 	8550 2800 8900 2800
