File: kicad/stm32l053c.sch (KiCad schematic (older format))
At the start: 36 parts, among them P1 SWD, P2 PWR, Q1 Q_PNP_BEC, SW1 SW_PUSH, SW2 SW_PUSH, SW3 SW_PUSH, U1 STM32L053C8_LQFP48, U2 TLV61225, U3 um66t, Y1 Crystal

Commit message: Buzzer transistor to be decided
Parts:
- removed Q1: Q_PNP_BEC, TO_SOT_Packages_SMD:SOT-23_Handsoldering, symbol Q_PNP_BEC
- removed R8: 10K, Resistors_SMD:R_0805_HandSoldering, symbol R
Connections:
- wire segments 112 -> 93
Other:
- moved on the sheet: D4, DS1, LS1
Changed lines of the file:
@@
 OSC32_OUT
 NoConn ~ 4600 4700
-Text Label 8700 4650 0    60   ~ 0
+Text Label 8850 1400 0    60   ~ 0
 LCD_COM0
-Text Label 8700 4750 0    60   ~ 0
+Text Label 8850 1500 0    60   ~ 0
 LCD_COM1
-Text Label 8700 4850 0    60   ~ 0
+Text Label 8850 1600 0    60   ~ 0
 LCD_COM2
-Text Label 8700 5150 0    60   ~ 0
+Text Label 8850 1900 0    60   ~ 0
 LCD_SEG0
-Text Label 8700 5250 0    60   ~ 0
+Text Label 8850 2000 0    60   ~ 0
 LCD_SEG1
-Text Label 8700 5350 0    60   ~ 0
+Text Label 8850 2100 0    60   ~ 0
 LCD_SEG2
-Text Label 8700 5450 0    60   ~ 0
+Text Label 8850 2200 0    60   ~ 0
 LCD_SEG3
-Text Label 8700 5550 0    60   ~ 0
+Text Label 8850 2300 0    60   ~ 0
 LCD_SEG4
-Text Label 8700 5650 0    60   ~ 0
+Text Label 8850 2400 0    60   ~ 0
 LCD_SEG5
-Text Label 8700 5750 0    60   ~ 0
+Text Label 8850 2500 0    60   ~ 0
 LCD_SEG6
-Text Label 8700 5850 0    60   ~ 0
+Text Label 8850 2600 0    60   ~ 0
 LCD_SEG7
-Text Label 8700 4950 0    60   ~ 0
+Text Label 8850 1700 0    60   ~ 0
 LCD_COM3
 $Comp
 L LCD_KITCHEN_TIMER DS1
 U 1 1 584F1C3C
-P 9700 5250
-F 0 "DS1" V 9700 5500 60  0000 C CNN
-F 1 "LCD_KITCHEN_TIMER" H 9700 5350 60  0000 C CNN
-F 2 "theapi:ZEBRA-12" H 9700 5250 60  0001 C CNN
-F 3 "" H 9700 5250 60  0000 C CNN
-	1    9700 5250
+P 9850 2000
+F 0 "DS1" V 9850 2250 60  0000 C CNN
+F 1 "LCD_KITCHEN_TIMER" H 9850 2100 60  0000 C CNN
+F 2 "theapi:ZEBRA-12" H 9850 2000 60  0001 C CNN
+F 3 "" H 9850 2000 60  0000 C CNN
+	1    9850 2000
 	0    1    1    0
 $EndComp
@@
 L BUZZER LS1
 U 1 1 5851ABB3
-P 9100 2950
-F 0 "LS1" H 9100 3200 60  0000 C CNN
-F 1 "BUZZER" H 9500 2950 60  0000 C CNN
-F 2 "Resistors_SMD:R_0805_HandSoldering" H 9250 3200 60  0001 C CNN
-F 3 "" H 9250 3200 60  0001 C CNN
-	1    9100 2950
+P 9100 4150
+F 0 "LS1" H 9100 4400 60  0000 C CNN
+F 1 "BUZZER" H 9500 4150 60  0000 C CNN
+F 2 "Resistors_SMD:R_0805_HandSoldering" H 9250 4400 60  0001 C CNN
+F 3 "" H 9250 4400 60  0001 C CNN
+	1    9100 4150
 	1    0    0    -1
 $EndComp
@@
 L Earth #PWR025
 U 1 1 5851B22D
-P 8900 3850
-F 0 "#PWR025" H 8900 3600 50  0001 C CNN
-F 1 "Earth" H 8900 3700 50  0001 C CNN
-F 2 "" H 8900 3850 50  0000 C CNN
-F 3 "" H 8900 3850 50  0000 C CNN
-	1    8900 3850
+P 8900 4850
+F 0 "#PWR025" H 8900 4600 50  0001 C CNN
+F 1 "Earth" H 8900 4700 50  0001 C CNN
+F 2 "" H 8900 4850 50  0000 C CNN
+F 3 "" H 8900 4850 50  0000 C CNN
+	1    8900 4850
 	1    0    0    -1
 $EndComp
@@
 Text Label 2600 2300 0    60   ~ 0
 BUTTON2
-$Comp
-L Q_PNP_BEC Q1
-U 1 1 586901C2
-P 8800 3650
-F 0 "Q1" H 9000 3700 50  0000 L CNN
-F 1 "Q_PNP_BEC" H 9000 3600 50  0000 L CNN
-F 2 "TO_SOT_Packages_SMD:SOT-23_Handsoldering" H 9000 3750 50  0001 C CNN
-F 3 "" H 8800 3650 50  0000 C CNN
-	1    8800 3650
-	1    0    0    -1
-$EndComp
 Text Label 7100 3500 2    60   ~ 0
 MELODY
@@
 Connection ~ 5450 5650
 Wire Wire Line
-	5450 1050 5450 1250
-Wire Wire Line
-	5450 1250 5450 2000
+	5450 1050 5450 2000
 Wire Wire Line
 	5550 1250 5550 2000
@@
 	5300 1250 5300 2000
 Wire Wire Line
-	5300 1250 5450 1250
-Wire Wire Line
-	5450 1250 5550 1250
-Wire Wire Line
-	5550 1250 5900 1250
+	5300 1250 5900 1250
 Connection ~ 5450 1250
 Wire Wire Line
@@
 	6550 2600 7100 2600
 Wire Wire Line
-	5450 5650 5550 5650
-Wire Wire Line
-	5550 5650 5650 5650
+	5450 5650 5650 5650
 Wire Wire Line
 	3450 4800 4600 4800
 Wire Wire Line
-	3450 4800 3450 5050
-Wire Wire Line
-	3450 5050 3450 5250
+	3450 4800 3450 5250
 Connection ~ 3450 5050
 Wire Wire Line
 	3750 4900 4600 4900
 Wire Wire Line
-	3750 4900 3750 5050
-Wire Wire Line
-	3750 5050 3750 5250
+	3750 4900 3750 5250
 Connection ~ 3750 5050
 Wire Wire Line
 	3750 5700 3750 5550
 Wire Wire Line
-	3450 5700 3600 5700
-Wire Wire Line
-	3600 5700 3750 5700
+	3450 5700 3750 5700
 Wire Wire Line
 	3450 5550 3450 5700
 Connection ~ 3600 5700
 Wire Wire Line
-	850  6750 1100 6750
-Wire Wire Line
-	1100 6750 1250 6750
-Wire Wire Line
-	1250 6750 1600 6750
-Wire Wire Line
-	1600 6750 1700 6750
+	850  6750 1700 6750
 Connection ~ 1250 6750
 Wire Wire Line
@@
 Connection ~ 1600 6750
 Wire Wire Line
-	2600 6550 2700 6550
-Wire Wire Line
-	2700 6550 2850 6550
-Wire Wire Line
-	2850 6550 3100 6550
+	2600 6550 3100 6550
 Connection ~ 2850 6550
 Wire Wire Line
@@
 Connection ~ 2700 6550
 Wire Wire Line
-	8700 4650 9250 4650
-Wire Wire Line
-	9250 4750 8700 4750
-Wire Wire Line
-	8700 4850 9250 4850
-Wire Wire Line
-	8700 4950 9250 4950
-Wire Wire Line
-	8700 5150 9250 5150
-Wire Wire Line
-	8700 5250 9250 5250
-Wire Wire Line
-	8700 5350 9250 5350
-Wire Wire Line
-	8700 5450 9250 5450
-Wire Wire Line
-	8700 5550 9250 5550
-Wire Wire Line
-	8700 5650 9250 5650
-Wire Wire Line
-	8700 5750 9250 5750
-Wire Wire Line
-	8700 5850 9250 5850
+	8850 1400 9400 1400
+Wire Wire Line
+	9400 1500 8850 1500
+Wire Wire Line
+	8850 1600 9400 1600
+Wire Wire Line
+	8850 1700 9400 1700
+Wire Wire Line
+	8850 1900 9400 1900
+Wire Wire Line
+	8850 2000 9400 2000
+Wire Wire Line
+	8850 2100 9400 2100
+Wire Wire Line
+	8850 2200 9400 2200
+Wire Wire Line
+	8850 2300 9400 2300
+Wire Wire Line
+	8850 2400 9400 2400
+Wire Wire Line
+	8850 2500 9400 2500
+Wire Wire Line
+	8850 2600 9400 2600
 Wire Wire Line
 	1300 2700 1300 2850
@@
 	2450 2850 3000 2850
 Wire Wire Line
-	8900 3000 8900 3100
-Wire Wire Line
-	8900 3100 8900 3450
+	8900 4200 8900 4650
 Wire Wire Line
 	8600 3650 8500 3650
 Wire Wire Line
-	8200 3650 8100 3650
-Wire Wire Line
-	8100 3650 7700 3650
+	7700 3650 8200 3650
 Wire Wire Line
 	3400 6550 3700 6550
@@
 	2600 1700 3200 1700
 Wire Wire Line
-	3500 2300 3800 2300
-Wire Wire Line
-	3800 2300 4600 2300
+	3500 2300 4600 2300
 Wire Wire Line
 	3500 1700 3800 1700
 Wire Wire Line
-	3800 1700 3800 2000
-Wire Wire Line
-	3800 2000 3800 2300
+	3800 1700 3800 2300
 Wire Wire Line
 	3500 2000 3800 2000
@@
 $EndComp
 Wire Wire Line
-	7700 4000 7700 4000
-Wire Wire Line
-	7700 3400 7700 3650
-Wire Wire Line
-	7700 3650 7700 4000
+	7700 3400 7700 4000
 Connection ~ 7700 3650
 Text Notes 6750 4350 0    60   ~ 0
@@
 L D D4
 U 1 1 586A5FCA
-P 8550 2950
-F 0 "D4" H 8550 3050 50  0000 C CNN
-F 1 "D" H 8550 2850 50  0000 C CNN
-F 2 "Diodes_SMD:D_0805" H 8550 2950 50  0001 C CNN
-F 3 "" H 8550 2950 50  0000 C CNN
-	1    8550 2950
-	0    1    1    0
-$EndComp
-Wire Wire Line
-	8900 2900 8900 2800
-Wire Wire Line
-	8900 2800 8900 2650
-Wire Wire Line
-	8550 2800 8900 2800
-Connection ~ 8900 2800
-Wire Wire Line
-	8550 3100 8900 3100
-Connection ~ 8900 3100
+P 8550 4150
+F 0 "D4" H 8550 4250 50  0000 C CNN
+F 1 "D" H 8550 4050 50  0000 C CNN
+F 2 "Diodes_SMD:D_0805" H 8550 4150 50  0001 C CNN
+F 3 "" H 8550 4150 50  0000 C CNN
+	1    8550 4150
+	0    1    1    0
+$EndComp
+Wire Wire Line
+	8900 3850 8900 4100
+Wire Wire Line
+	8550 4000 8900 4000
+Connection ~ 8900 4000
+Wire Wire Line
+	8550 4300 8900 4300
+Connection ~ 8900 4300
 $Comp
 L +BATT #PWR029
 U 1 1 586A907B
-P 8900 2650
-F 0 "#PWR029" H 8900 2500 50  0001 C CNN
-F 1 "+BATT" H 8900 2790 50  0000 C CNN
-F 2 "" H 8900 2650 50  0000 C CNN
-F 3 "" H 8900 2650 50  0000 C CNN
-	1    8900 2650
+P 8900 3350
+F 0 "#PWR029" H 8900 3200 50  0001 C CNN
+F 1 "+BATT" H 8900 3490 50  0000 C CNN
+F 2 "" H 8900 3350 50  0000 C CNN
+F 3 "" H 8900 3350 50  0000 C CNN
+	1    8900 3350
 	1    0    0    -1
 $EndComp
 Wire Wire Line
 	6550 3500 7100 3500
-$Comp
-L R R8
-U 1 1 586AB55A
-P 8100 3900
-F 0 "R8" V 8180 3900 50  0000 C CNN
-F 1 "10K" V 8100 3900 50  0000 C CNN
-F 2 "Resistors_SMD:R_0805_HandSoldering" V 8030 3900 50  0001 C CNN
-F 3 "" H 8100 3900 50  0000 C CNN
-	1    8100 3900
-	-1   0    0    1
-$EndComp
 Wire Wire Line
 	7100 3500 7100 3800
-$Comp
-L Earth #PWR?
-U 1 1 586AC8CF
-P 8100 4050
-F 0 "#PWR?" H 8100 3800 50  0001 C CNN
-F 1 "Earth" H 8100 3900 50  0001 C CNN
-F 2 "" H 8100 4050 50  0000 C CNN
-F 3 "" H 8100 4050 50  0000 C CNN
-	1    8100 4050
-	1    0    0    -1
-$EndComp
-Wire Wire Line
-	8100 3750 8100 3650
-Connection ~ 8100 3650
+Wire Wire Line
+	8900 3450 8900 3350
 $EndSCHEMATC

Commit message: BC817 transistor
Parts:
- added Q?: BC817, SOT-23, symbol BC817-40
- added R?: 0, Resistors_SMD:R_0805_HandSoldering, symbol R
Changed lines of the file:
@@
 	5550 1250 5550 2000
-Wire Wire Line
-	5300 1250 5300 2000
 Wire Wire Line
 	5300 1250 5900 1250
@@
 Wire Wire Line
 	8900 3450 8900 3350
+$Comp
+L BC817-40 Q?
+U 1 1 586BB01F
+P 8800 3650
+F 0 "Q?" H 9000 3725 50  0000 L CNN
+F 1 "BC817" H 9000 3650 50  0000 L CNN
+F 2 "SOT-23" H 9000 3575 50  0000 L CIN
+F 3 "" H 8800 3650 50  0000 L CNN
+	1    8800 3650
+	1    0    0    -1
+$EndComp
+$Comp
+L R R?
+U 1 1 586BB489
+P 5300 1400
+F 0 "R?" V 5380 1400 50  0000 C CNN
+F 1 "0" V 5300 1400 50  0000 C CNN
+F 2 "Resistors_SMD:R_0805_HandSoldering" V 5230 1400 50  0001 C CNN
+F 3 "" H 5300 1400 50  0000 C CNN
+	1    5300 1400
+	-1   0    0    1
+$EndComp
+Wire Wire Line
+	5300 1550 5300 2000
 $EndSCHEMATC

Commit message: PNP & more layout
Parts:
- removed D4: D, Diodes_SMD:D_0805, symbol D
- removed Q?: BC817, SOT-23, symbol BC817-40
- added Q1: BC807, TO_SOT_Packages_SMD:SOT-23_Handsoldering, symbol BC807-40
- D1, D2, D3: footprint Diodes_SMD:D_0805 -> Diodes_SMD:SOD-523
- U2: footprint TO_SOT_Packages_SMD:SC-70-6 -> theapi:SC-70-6
- gave numbers to parts that had none: 1
Connections:
- net +BATT: now also Q1.2 (E)
- net Earth: now also LS1.2 (-)
- net at LS1.1 (+): now also Q1.3 (C)
- net at R6.1: now also Q1.1 (B)
Changed lines of the file:
@@
 F 0 "U2" H 2150 6650 60  0000 C CNN
 F 1 "TLV61225" H 2150 5950 60  0000 C CNN
-F 2 "TO_SOT_Packages_SMD:SC-70-6" H 2150 6550 60  0001 C CNN
+F 2 "theapi:SC-70-6" H 2150 6550 60  0001 C CNN
 F 3 "" H 2150 6550 60  0001 C CNN
 	1    2150 6500
@@
 L Earth #PWR025
 U 1 1 5851B22D
-P 8900 4850
-F 0 "#PWR025" H 8900 4600 50  0001 C CNN
-F 1 "Earth" H 8900 4700 50  0001 C CNN
-F 2 "" H 8900 4850 50  0000 C CNN
-F 3 "" H 8900 4850 50  0000 C CNN
-	1    8900 4850
+P 8900 4650
+F 0 "#PWR025" H 8900 4400 50  0001 C CNN
+F 1 "Earth" H 8900 4500 50  0001 C CNN
+F 2 "" H 8900 4650 50  0000 C CNN
+F 3 "" H 8900 4650 50  0000 C CNN
+	1    8900 4650
 	1    0    0    -1
 $EndComp
@@
 F 0 "D3" H 3350 2400 50  0000 C CNN
 F 1 "D_Schottky" H 3350 2200 50  0000 C CNN
-F 2 "Diodes_SMD:D_0805" H 3350 2300 50  0001 C CNN
+F 2 "Diodes_SMD:SOD-523" H 3350 2300 50  0001 C CNN
 F 3 "" H 3350 2300 50  0000 C CNN
 	1    3350 2300
@@
 F 0 "D2" H 3350 2100 50  0000 C CNN
 F 1 "D_Schottky" H 3350 1900 50  0000 C CNN
-F 2 "Diodes_SMD:D_0805" H 3350 2000 50  0001 C CNN
+F 2 "Diodes_SMD:SOD-523" H 3350 2000 50  0001 C CNN
 F 3 "" H 3350 2000 50  0000 C CNN
 	1    3350 2000
@@
 F 0 "D1" H 3350 1800 50  0000 C CNN
 F 1 "D_Schottky" H 3350 1600 50  0000 C CNN
-F 2 "Diodes_SMD:D_0805" H 3350 1700 50  0001 C CNN
+F 2 "Diodes_SMD:SOD-523" H 3350 1700 50  0001 C CNN
 F 3 "" H 3350 1700 50  0000 C CNN
 	1    3350 1700
@@
 Text Notes 6750 4350 0    60   ~ 0
 Either BUZZER or MELODY
-$Comp
-L D D4
-U 1 1 586A5FCA
-P 8550 4150
-F 0 "D4" H 8550 4250 50  0000 C CNN
-F 1 "D" H 8550 4050 50  0000 C CNN
-F 2 "Diodes_SMD:D_0805" H 8550 4150 50  0001 C CNN
-F 3 "" H 8550 4150 50  0000 C CNN
-	1    8550 4150
-	0    1    1    0
-$EndComp
 Wire Wire Line
 	8900 3850 8900 4100
-Wire Wire Line
-	8550 4000 8900 4000
-Connection ~ 8900 4000
-Wire Wire Line
-	8550 4300 8900 4300
-Connection ~ 8900 4300
 $Comp
 L +BATT #PWR029
@@
 	8900 3450 8900 3350
 $Comp
-L BC817-40 Q?
-U 1 1 586BB01F
-P 8800 3650
-F 0 "Q?" H 9000 3725 50  0000 L CNN
-F 1 "BC817" H 9000 3650 50  0000 L CNN
-F 2 "SOT-23" H 9000 3575 50  0000 L CIN
-F 3 "" H 8800 3650 50  0000 L CNN
-	1    8800 3650
-	1    0    0    -1
-$EndComp
-$Comp
-L R R?
+L R R8
 U 1 1 586BB489
 P 5300 1400
-F 0 "R?" V 5380 1400 50  0000 C CNN
+F 0 "R8" V 5380 1400 50  0000 C CNN
 F 1 "0" V 5300 1400 50  0000 C CNN
 F 2 "Resistors_SMD:R_0805_HandSoldering" V 5230 1400 50  0001 C CNN
@@
 Wire Wire Line
 	5300 1550 5300 2000
+$Comp
+L BC807-40 Q1
+U 1 1 586C1223
+P 8800 3650
+F 0 "Q1" H 9000 3725 50  0000 L CNN
+F 1 "BC807" H 9000 3650 50  0000 L CNN
+F 2 "TO_SOT_Packages_SMD:SOT-23_Handsoldering" H 9000 3575 50  0000 L CIN
+F 3 "" H 8800 3650 50  0000 L CNN
+	1    8800 3650
+	1    0    0    1
+$EndComp
 $EndSCHEMATC
