File: kicad/stm32l053c.kicad_pcb (KiCad board)
At the start: 2 copper layers, 52 x 36 mm, 47 parts, among them P1 SWD, P2 PWR, Q1 BC807, Q2 BC817, SW1 SW_PUSH, SW2 SW_PUSH, SW3 SW_PUSH, SW4 SW_SPDT, U1 STM32L053C8_LQFP48, U2 TLV61225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

Commit message: Labels
Parts:
- renumbered W1 to PA5
Changed lines of the file:
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@@
     (area 116.924999 84.524999 169.075001 120.675001)
     (thickness 1.6)
-    (drawings 25)
+    (drawings 32)
     (tracks 556)
     (zones 0)
@@
   (layers
     (0 F.Cu signal)
-    (31 B.Cu signal)
+    (31 B.Cu signal hide)
     (32 B.Adhes user)
     (33 F.Adhes user)
@@
     (solder_mask_margin 0.07)
     (attr smd)
-    (fp_text reference U2 (at 0.01016 3.05054 180) (layer B.SilkS)
+    (fp_text reference U2 (at -1.505807 -2.548581 180) (layer B.SilkS)
       (effects (font (size 1 1) (thickness 0.15)) (justify mirror))
     )
@@
     (solder_mask_margin 0.07)
     (attr smd)
-    (fp_text reference U1 (at 0 -6) (layer F.SilkS)
+    (fp_text reference U1 (at 0 0) (layer F.SilkS)
       (effects (font (size 1 1) (thickness 0.15)))
     )
@@
     (tags "capacitor 0805")
     (attr smd)
-    (fp_text reference C4 (at 3.366535 -0.180312 180) (layer B.SilkS)
+    (fp_text reference C4 (at 0 2.1 180) (layer B.SilkS)
       (effects (font (size 1 1) (thickness 0.15)) (justify mirror))
     )
@@
     (tags "capacitor 0805")
     (attr smd)
-    (fp_text reference C5 (at -3.412497 0 180) (layer B.SilkS)
+    (fp_text reference C5 (at 0 -3.75 180) (layer B.SilkS)
       (effects (font (size 1 1) (thickness 0.15)) (justify mirror))
     )
@@
     (tags "capacitor 0603")
     (attr smd)
-    (fp_text reference C8 (at 0 1.9 270) (layer B.SilkS)
+    (fp_text reference C8 (at -1.051419 1.094193 270) (layer B.SilkS)
       (effects (font (size 1 1) (thickness 0.15)) (justify mirror))
     )
@@
     (tags "capacitor 0603")
     (attr smd)
-    (fp_text reference C9 (at 0 1.9 270) (layer B.SilkS)
+    (fp_text reference C9 (at 0.748581 -1.405807 270) (layer B.SilkS)
       (effects (font (size 1 1) (thickness 0.15)) (justify mirror))
     )
@@
     (tags "resistor 0805")
     (attr smd)
-    (fp_text reference R2 (at 0 2.1 180) (layer B.SilkS)
+    (fp_text reference R2 (at -0.05 1.7 180) (layer B.SilkS)
       (effects (font (size 1 1) (thickness 0.15)) (justify mirror))
     )
@@
     (tags "resistor 0805")
     (attr smd)
-    (fp_text reference R3 (at 0 2.1 180) (layer B.SilkS)
+    (fp_text reference R3 (at 0 3.75 180) (layer B.SilkS)
       (effects (font (size 1 1) (thickness 0.15)) (justify mirror))
     )
@@
     (tags "resistor 0805")
     (attr smd)
-    (fp_text reference R6 (at 0 -1.794193) (layer F.SilkS)
+    (fp_text reference R6 (at 0 1.8) (layer F.SilkS)
       (effects (font (size 1 1) (thickness 0.15)))
     )
@@
     (tags "inductor taiyo-yuden nr smd")
     (attr smd)
-    (fp_text reference L1 (at 0 2.5 180) (layer B.SilkS)
+    (fp_text reference L1 (at 3.694193 -0.048581 180) (layer B.SilkS)
       (effects (font (size 1 1) (thickness 0.15)) (justify mirror))
     )
@@
     (tags Switch)
     (attr smd)
-    (fp_text reference SW2 (at 0 -6 180) (layer F.SilkS)
+    (fp_text reference SW2 (at 0 -6 180) (layer Cmts.User)
       (effects (font (size 1 1) (thickness 0.15)))
     )
@@
     (tags Switch)
     (attr smd)
-    (fp_text reference SW1 (at 0 -6 180) (layer F.SilkS)
+    (fp_text reference SW1 (at 0 -6 180) (layer Cmts.User)
       (effects (font (size 1 1) (thickness 0.15)))
     )
@@
   (module theapi:ZEBRA-12 locked (layer F.Cu)
     (at 143 101)
-    (fp_text reference DS1 (at 0 3.2) (layer F.SilkS)
+    (fp_text reference DS1 (at 0 3.2) (layer Cmts.User)
       (effects (font (size 1.2 1.2) (thickness 0.15)))
     )
@@
     (tags Switch)
     (attr smd)
-    (fp_text reference SW3 (at 0 -6 180) (layer F.SilkS)
+    (fp_text reference SW3 (at 0 -6 180) (layer Cmts.User)
       (effects (font (size 1 1) (thickness 0.15)))
     )
@@
     (tags "Diode SOD523")
     (attr smd)
-    (fp_text reference D3 (at 0 1.5 270) (layer B.SilkS)
+    (fp_text reference D3 (at 0.05 -1.5 270) (layer B.SilkS)
       (effects (font (size 1 1) (thickness 0.15)) (justify mirror))
     )
@@
     (tags SOT-23)
     (attr smd)
-    (fp_text reference Q2 (at 0 -2.5 270) (layer F.SilkS)
+    (fp_text reference Q2 (at 3.5 0 360) (layer F.SilkS)
       (effects (font (size 1 1) (thickness 0.15)))
     )
@@
     (tags "resistor 0805")
     (attr smd)
-    (fp_text reference R9 (at 0 -2.1) (layer F.SilkS)
+    (fp_text reference R9 (at 0 -1.55) (layer F.SilkS)
       (effects (font (size 1 1) (thickness 0.15)))
     )
@@
     (tags "capacitor 0603")
     (attr smd)
-    (fp_text reference C6 (at 0 -1.9 180) (layer F.SilkS)
+    (fp_text reference C6 (at 0.4 -1.6 180) (layer F.SilkS)
       (effects (font (size 1 1) (thickness 0.15)))
     )
@@
     (tags "capacitor 0603")
     (attr smd)
-    (fp_text reference C7 (at 0 -1.9 180) (layer F.SilkS)
+    (fp_text reference C7 (at 0.4 1.4 180) (layer F.SilkS)
       (effects (font (size 1 1) (thickness 0.15)))
     )
@@
     (tags "resistor 0805")
     (attr smd)
-    (fp_text reference R10 (at 0 -2.1) (layer F.SilkS)
+    (fp_text reference R10 (at 0 1.55) (layer F.SilkS)
       (effects (font (size 1 1) (thickness 0.15)))
     )
@@
     (tags "SMD SMT crystal hand-soldering")
     (attr smd)
-    (fp_text reference Y1 (at 0 4.5 180) (layer B.SilkS)
+    (fp_text reference Y1 (at 0.1 0 180) (layer B.SilkS)
       (effects (font (size 1 1) (thickness 0.15)) (justify mirror))
     )
@@
     (tags "Mesurement Point Round Trough Hole 1.5mm Drill 0.8mm")
     (attr virtual)
-    (fp_text reference W1 (at 0 -2) (layer F.SilkS)
+    (fp_text reference PA5 (at 0 2) (layer F.SilkS)
       (effects (font (size 1 1) (thickness 0.15)))
     )
@@
     (descr "Through hole straight pin header, 1x03, 2.54mm pitch, single row")
     (tags "Through hole pin header THT 1x03 2.54mm single row")
-    (fp_text reference SW4 (at 0 -2.39 270) (layer F.SilkS)
+    (fp_text reference SW4 (at 0 -2.39 270) (layer Cmts.User)
       (effects (font (size 1 1) (thickness 0.15)))
     )
@@
       (xy 11.555941 15.398411)) (layer B.SilkS) (width 0.01))
   )
+  (gr_text NRST (at 132 87.6 360) (layer F.SilkS)
+    (effects (font (size 0.8 0.8) (thickness 0.15)))
+  )
+  (gr_text SWDIO (at 126.6 91 270) (layer F.SilkS)
+    (effects (font (size 0.8 0.8) (thickness 0.15)))
+  )
+  (gr_text GND (at 124.05 90.75 270) (layer F.SilkS)
+    (effects (font (size 0.8 0.8) (thickness 0.15)))
+  )
+  (gr_text SWCLK (at 121.5 91.3 270) (layer F.SilkS)
+    (effects (font (size 0.8 0.8) (thickness 0.15)))
+  )
+  (gr_text VDD (at 119 90.5 270) (layer F.SilkS)
+    (effects (font (size 0.8 0.8) (thickness 0.15)))
+  )
+  (gr_text - (at 165.6 96.2) (layer B.SilkS)
+    (effects (font (size 0.8 0.8) (thickness 0.15)) (justify mirror))
+  )
+  (gr_text + (at 165.5 93.6) (layer B.SilkS)
+    (effects (font (size 0.8 0.8) (thickness 0.15)) (justify mirror))
+  )
   (dimension 52 (width 0.15) (layer Dwgs.User)
     (gr_text "52.000 mm" (at 143 79.9) (layer Dwgs.User)
@@
   (gr_line (start 117 84.6) (end 117 85.6) (layer Edge.Cuts) (width 0.15))
   (gr_line (start 169 84.6) (end 169 85.6) (layer Edge.Cuts) (width 0.15))
-  (gr_text NRST (at 129.3 91 270) (layer B.SilkS)
+  (gr_text NRST (at 130.4 89.8) (layer B.SilkS)
     (effects (font (size 0.8 0.8) (thickness 0.15)) (justify mirror))
   )
@@
     (effects (font (size 0.8 0.8) (thickness 0.15)) (justify mirror))
   )
-  (gr_text SWDIO (at 126.55 91.05 270) (layer B.SilkS)
+  (gr_text SWDIO (at 126.2 91 270) (layer B.SilkS)
     (effects (font (size 0.8 0.8) (thickness 0.15)) (justify mirror))
   )
-  (gr_text + (at 165.8 93.8) (layer F.SilkS)
+  (gr_text + (at 165.5 93.6) (layer F.SilkS)
     (effects (font (size 0.8 0.8) (thickness 0.15)))
   )

Commit message: Labels
Parts:
- Melody or Buzzer: renamed from R1
- PWR SB: renamed from R7
- moved G*** 3.80 mm to (148.9, 108.4)
- renumbered P2 to BAT, Q2 to NPN, Q1 to PNP, SW4 to SW_VOL
Other:
- board text added: "LOUD"
- board text added: "PA5"
- board text added: "QUIET"
Changed lines of the file:
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@@
     (links 113)
     (no_connects 0)
-    (area 116.924999 84.524999 169.075001 120.675001)
+    (area 107.214285 79.2 185.166669 135.515001)
     (thickness 1.6)
-    (drawings 32)
+    (drawings 35)
     (tracks 556)
     (zones 0)
@@
   (layers
     (0 F.Cu signal)
-    (31 B.Cu signal hide)
+    (31 B.Cu signal)
     (32 B.Adhes user)
     (33 F.Adhes user)
@@
     (38 B.Mask user)
     (39 F.Mask user)
-    (40 Dwgs.User user)
+    (40 Dwgs.User user hide)
     (41 Cmts.User user)
     (42 Eco1.User user)
@@
     (solder_mask_margin 0.07)
     (attr smd)
-    (fp_text reference U2 (at -1.505807 -2.548581 180) (layer B.SilkS)
-      (effects (font (size 1 1) (thickness 0.15)) (justify mirror))
+    (fp_text reference U2 (at -1.505807 -2.548581 180) (layer Cmts.User)
+      (effects (font (size 1 1) (thickness 0.15)))
     )
     (fp_text value TLV61225 (at 0.04064 -4.191 180) (layer B.Fab)
@@
     (tags "resistor 0805")
     (attr smd)
-    (fp_text reference R7 (at 0 2.1) (layer B.SilkS)
-      (effects (font (size 1 1) (thickness 0.15)) (justify mirror))
+    (fp_text reference "PWR SB" (at -0.6 3.25 90) (layer B.SilkS)
+      (effects (font (size 0.8 0.8) (thickness 0.15)) (justify mirror))
     )
     (fp_text value 0 (at 0 -2.1) (layer B.Fab)
@@
     (descr "Through hole pin header")
     (tags "pin header")
-    (fp_text reference P1 (at 0 3 270) (layer B.SilkS)
-      (effects (font (size 1 1) (thickness 0.15)) (justify mirror))
+    (fp_text reference P1 (at 0 3 270) (layer Cmts.User)
+      (effects (font (size 1 1) (thickness 0.15)))
     )
     (fp_text value SWD (at 0 3.1 270) (layer B.Fab)
@@
     (tags "capacitor 0805")
     (attr smd)
-    (fp_text reference C1 (at 0.02 -1.778) (layer B.SilkS)
+    (fp_text reference C1 (at 3.2 0 180) (layer B.SilkS)
       (effects (font (size 1 1) (thickness 0.15)) (justify mirror))
     )
@@
     (tags "capacitor 0805")
     (attr smd)
-    (fp_text reference C2 (at -0.02 1.778 90) (layer B.SilkS)
+    (fp_text reference C2 (at -1.2 -1.9 180) (layer B.SilkS)
       (effects (font (size 1 1) (thickness 0.15)) (justify mirror))
     )
@@
     (tags "capacitor 0805")
     (attr smd)
-    (fp_text reference C3 (at -3.312795 0.081317 90) (layer B.SilkS)
+    (fp_text reference C3 (at -1.3 1.9 180) (layer B.SilkS)
       (effects (font (size 1 1) (thickness 0.15)) (justify mirror))
     )
@@
     (tags "capacitor 0805")
     (attr smd)
-    (fp_text reference C4 (at 0 2.1 180) (layer B.SilkS)
+    (fp_text reference C4 (at -0.1 1.7 180) (layer B.SilkS)
       (effects (font (size 1 1) (thickness 0.15)) (justify mirror))
     )
@@
     (tags "resistor 0805")
     (attr smd)
-    (fp_text reference R4 (at 0 -1.651 180) (layer B.SilkS)
+    (fp_text reference R4 (at 3.5 0 180) (layer B.SilkS)
       (effects (font (size 1 1) (thickness 0.15)) (justify mirror))
     )
@@
     (tags "capacitor 0603")
     (attr smd)
-    (fp_text reference C8 (at -1.051419 1.094193 270) (layer B.SilkS)
+    (fp_text reference C8 (at 0.048581 1.794193 360) (layer B.SilkS)
       (effects (font (size 1 1) (thickness 0.15)) (justify mirror))
     )
@@
     (tags "capacitor 0603")
     (attr smd)
-    (fp_text reference C9 (at 0.748581 -1.405807 270) (layer B.SilkS)
+    (fp_text reference C9 (at 1.148581 -1.605807 360) (layer B.SilkS)
       (effects (font (size 1 1) (thickness 0.15)) (justify mirror))
     )
@@
     (tags "capacitor 0805")
     (attr smd)
-    (fp_text reference C10 (at 0 2.1 180) (layer B.SilkS)
+    (fp_text reference C10 (at 3.9 0 180) (layer B.SilkS)
       (effects (font (size 1 1) (thickness 0.15)) (justify mirror))
     )
@@
     (tags "capacitor 0805")
     (attr smd)
-    (fp_text reference C11 (at 0 2.1) (layer B.SilkS)
+    (fp_text reference C11 (at 0 3.7) (layer B.SilkS)
       (effects (font (size 1 1) (thickness 0.15)) (justify mirror))
     )
@@
     (tags "resistor 0805")
     (attr smd)
-    (fp_text reference LS1 (at 0 2.1 270) (layer B.SilkS)
+    (fp_text reference LS1 (at -3.1 0 360) (layer B.SilkS)
       (effects (font (size 1 1) (thickness 0.15)) (justify mirror))
     )
@@
     (tags SOT-23)
     (attr smd)
-    (fp_text reference Q1 (at -0.198581 1.294193 90) (layer B.SilkS)
+    (fp_text reference PNP (at -3.4 0 180) (layer B.SilkS)
       (effects (font (size 1 1) (thickness 0.15)) (justify mirror))
     )
@@
     (tags "resistor 0805")
     (attr smd)
-    (fp_text reference R5 (at 0 -1.75) (layer B.SilkS)
+    (fp_text reference R5 (at 0.1 -3.5) (layer B.SilkS)
       (effects (font (size 1 1) (thickness 0.15)) (justify mirror))
     )
@@
     (descr "Through hole pin header")
     (tags "pin header")
-    (fp_text reference P2 (at 0 2 180) (layer B.SilkS)
-      (effects (font (size 1 1) (thickness 0.15)) (justify mirror))
+    (fp_text reference BAT (at 0 -4.6 180) (layer B.SilkS)
+      (effects (font (size 0.8 0.8) (thickness 0.15)) (justify mirror))
     )
     (fp_text value PWR (at 0 3.1 180) (layer B.Fab)
@@
     (tags "resistor 0805")
     (attr smd)
-    (fp_text reference R1 (at 0 2.1 270) (layer B.SilkS)
-      (effects (font (size 1 1) (thickness 0.15)) (justify mirror))
+    (fp_text reference "Melody or Buzzer" (at -2.9 -1.6 360) (layer B.SilkS)
+      (effects (font (size 0.7 0.7) (thickness 0.15)) (justify mirror))
     )
     (fp_text value 0 (at 0 -2.1 270) (layer B.Fab)
@@
     (tags "Diode SOD523")
     (attr smd)
-    (fp_text reference D1 (at 0 1.5 90) (layer B.SilkS)
+    (fp_text reference D1 (at 0 -1.7 180) (layer B.SilkS)
       (effects (font (size 1 1) (thickness 0.15)) (justify mirror))
     )
@@
     (tags "Diode SOD523")
     (attr smd)
-    (fp_text reference D2 (at 0 1.5 90) (layer B.SilkS)
-      (effects (font (size 1 1) (thickness 0.15)) (justify mirror))
+    (fp_text reference D2 (at 1.8 0.15 180) (layer B.SilkS)
+      (effects (font (size 0.8 0.8) (thickness 0.15)) (justify mirror))
     )
     (fp_text value D_Schottky (at 0 -1.7 90) (layer B.Fab)
@@
     (tags "Diode SOD523")
     (attr smd)
-    (fp_text reference D3 (at 0.05 -1.5 270) (layer B.SilkS)
+    (fp_text reference D3 (at 0 -1.7 360) (layer B.SilkS)
       (effects (font (size 1 1) (thickness 0.15)) (justify mirror))
     )
@@
     (tags SOT-23)
     (attr smd)
-    (fp_text reference Q2 (at 3.5 0 360) (layer F.SilkS)
+    (fp_text reference NPN (at 3.5 0 360) (layer F.SilkS)
       (effects (font (size 1 1) (thickness 0.15)))
     )
@@
     (descr "TO-92 leads in-line, narrow, oval pads, drill 0.6mm (see NXP sot054_po.pdf)")
     (tags "to-92 sc-43 sc-43a sot54 PA33 transistor")
-    (fp_text reference U3 (at 1.27 3.556) (layer B.SilkS)
-      (effects (font (size 1 1) (thickness 0.15)) (justify mirror))
+    (fp_text reference U3 (at 1.27 1.7) (layer Cmts.User)
+      (effects (font (size 1 1) (thickness 0.15)))
     )
     (fp_text value um66t (at 1.27 -2.794) (layer B.Fab)
@@
     (tags "Mesurement Point Round Trough Hole 1.5mm Drill 0.8mm")
     (attr virtual)
-    (fp_text reference PA5 (at 0 2) (layer F.SilkS)
-      (effects (font (size 1 1) (thickness 0.15)))
+    (fp_text reference PA5 (at -0.9 1.9 90) (layer B.SilkS)
+      (effects (font (size 0.8 0.8) (thickness 0.15)) (justify mirror))
     )
     (fp_text value TEST_1P (at 0 2) (layer F.Fab)
@@
     (descr "Through hole straight pin header, 1x03, 2.54mm pitch, single row")
     (tags "Through hole pin header THT 1x03 2.54mm single row")
-    (fp_text reference SW4 (at 0 -2.39 270) (layer Cmts.User)
-      (effects (font (size 1 1) (thickness 0.15)))
+    (fp_text reference SW_VOL (at -1.7 2.44 360) (layer B.SilkS)
+      (effects (font (size 0.8 0.8) (thickness 0.15)) (justify mirror))
     )
     (fp_text value SW_SPDT (at 0 7.47 270) (layer F.Fab)
@@
   )
   (module theapi:hero (layer B.Cu)
-    (at 149 104.6 180)
+    (at 148.9 108.4 180)
     (fp_text reference G*** (at 0 0 180) (layer B.SilkS) hide
       (effects (font (thickness 0.3)) (justify mirror))
@@
       (xy 11.555941 15.398411)) (layer B.SilkS) (width 0.01))
   )
-  (gr_text NRST (at 132 87.6 360) (layer F.SilkS)
+  (gr_text PA5 (at 145.8 105.6) (layer F.SilkS)
+    (effects (font (size 0.8 0.8) (thickness 0.15)))
+  )
+  (gr_text QUIET (at 164.8 89.7) (layer B.SilkS)
+    (effects (font (size 0.8 0.8) (thickness 0.15)) (justify mirror))
+  )
+  (gr_text LOUD (at 159.8 89.7) (layer B.SilkS)
+    (effects (font (size 0.8 0.8) (thickness 0.15)) (justify mirror))
+  )
+  (gr_text NRST (at 132 87.6) (layer F.SilkS)
     (effects (font (size 0.8 0.8) (thickness 0.15)))
   )
@@
     (arrow2b (pts (xy 117 80.6) (xy 118.126504 80.013579)))
   )
-  (gr_text "Peter Clarke" (at 141.5 113.6) (layer B.SilkS)
+  (gr_text "Peter Clarke" (at 142 117.6) (layer B.SilkS)
     (effects (font (size 1 1) (thickness 0.15)) (justify mirror))
   )
-  (gr_text "January 2017 v1.0" (at 141.5 111.6) (layer B.SilkS)
+  (gr_text "January 2017 v1.0" (at 142 115.6) (layer B.SilkS)
     (effects (font (size 0.8 0.8) (thickness 0.15) italic) (justify mirror))
   )
@@
     (arrow2b (pts (xy 176 120) (xy 175.413579 118.873496)))
   )
-  (gr_text github.com/theapi/kitchen_timer_stm32 (at 141.5 109.6) (layer B.SilkS)
+  (gr_text github.com/theapi/kitchen_timer_stm32 (at 142 113.6) (layer B.SilkS)
     (effects (font (size 0.8 0.8) (thickness 0.15)) (justify mirror))
   )
